File: Aidan PCB.kicad_pcb (KiCad board)
At the start: 2 copper layers, 82.1 x 38.8 mm, 24 parts, among them SW1 SW_Push, U1 ATmega32U4-AU, Y1 16MHz

Commit message: Updated schematic
Parts:
- moved D3 36.1 mm to (134.5, 80.9)
- moved D4 30.9 mm to (133.6, 70.6)
- moved D2 14.5 mm to (137.2, 90.7)
- moved D1 10.8 mm to (134.6, 98.1)
- moved C2 2.43 mm to (65.3, 81.7)
- moved R3 2.43 mm to (62.0, 81.7)
- moved C5 0.84 mm to (85.5, 89.3)
Routing:
- net Net-(R3-Pad2): track 0.00 -> 36.2 mm, vias 0 -> 2
- net ROW1: track 24.0 -> 0.00 mm
- net +5V: track 26.8 -> 49.5 mm
- net GND: track 144.2 -> 158.8 mm, vias 0 -> 2
- net Net-(D3-Pad2): track 7.71 -> 0.36 mm
Other:
- board size 82.1 x 38.8 mm -> 82.1 x 39 mm
