File: _autosave-Aidan PCB.kicad_pcb (KiCad board)
At the start: 2 copper layers, 82.1 x 38.8 mm, 24 parts, among them SW1 SW_Push, U1 ATmega32U4-AU, Y1 16MHz

Commit message: pcb tracing
Parts:
- moved C2 2.43 mm to (65.3, 81.7)
- moved R3 2.43 mm to (62.0, 81.7)
Routing:
- net Net-(R3-Pad2): track 0.00 -> 19.6 mm
- net +5V: track 26.8 -> 42.5 mm, vias 0 -> 7
- net (no net): vias 0 -> 1
Changed lines of the file:
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@@
     (thickness 1.6)
     (drawings 8)
-    (tracks 108)
+    (tracks 136)
     (zones 0)
     (modules 24)
@@
   )
   (module Capacitor_SMD:C_0805_2012Metric (layer B.Cu)
-    (at 65.925 84.075 270)
+    (at 65.3 81.725 270)
     (descr "Capacitor SMD 0805 (2012 Metric), square (rectangular) end terminal, IPC_7351 nominal, (Body size source: https://docs.google.com/spreadsheets/d/1BsfQQcO9C6DZCsRaXUlFlo91Tg2WpOkGARC1WS5S8t0/edit?usp=sharing), generated with kicad-footprint-generator")
     (tags capacitor)
@@
   )
   (module Resistor_SMD:R_0805_2012Metric (layer B.Cu)
-    (at 62.625 84.0625 270)
+    (at 62 81.7125 270)
     (descr "Resistor SMD 0805 (2012 Metric), square (rectangular) end terminal, IPC_7351 nominal, (Body size source: https://docs.google.com/spreadsheets/d/1BsfQQcO9C6DZCsRaXUlFlo91Tg2WpOkGARC1WS5S8t0/edit?usp=sharing), generated with kicad-footprint-generator")
     (tags resistor)
@@
   (gr_arc (start 123.515 73.91) (end 126.12 73.86) (angle -88.8) (layer Edge.Cuts) (width 0.5))
   (gr_arc (start 123.385 107.08) (end 123.275 109.75) (angle -94.07790525) (layer Edge.Cuts) (width 0.5))
+  (via (at 59.825 84.15) (size 0.8) (drill 0.4) (layers F.Cu B.Cu) (net 1))
+  (via (at 68.25 92.325) (size 0.8) (drill 0.4) (layers F.Cu B.Cu) (net 0))
+  (via (at 63.875 79.075) (size 0.8) (drill 0.4) (layers F.Cu B.Cu) (net 1))
+  (via (at 67.9 97.5) (size 0.8) (drill 0.4) (layers F.Cu B.Cu) (net 1))
+  (via (at 85.05 102.675) (size 0.8) (drill 0.4) (layers F.Cu B.Cu) (net 1))
+  (via (at 86.85 92.75) (size 0.8) (drill 0.4) (layers F.Cu B.Cu) (net 1))
+  (via (at 59.9 99.825) (size 0.8) (drill 0.4) (layers F.Cu B.Cu) (net 1))
   (segment (start 83 102.825) (end 83 101.15) (width 0.2032) (layer B.Cu) (net 1))
   (segment (start 83 101.15) (end 82.725 100.875) (width 0.2032) (layer B.Cu) (net 1))
@@
   (segment (start 57.018763 98.143763) (end 64.468763 98.143763) (width 0.2032) (layer B.Cu) (net 1))
   (segment (start 51.66071 92.78571) (end 57.018763 98.143763) (width 0.2032) (layer B.Cu) (net 1))
+  (segment (start 57.398399 98.523399) (end 57.018763 98.143763) (width 0.2032) (layer B.Cu) (net 1))
+  (segment (start 58.598399 98.523399) (end 57.398399 98.523399) (width 0.2032) (layer B.Cu) (net 1))
+  (segment (start 59.9 99.825) (end 58.598399 98.523399) (width 0.2032) (layer B.Cu) (net 1))
+  (via (at 67.9 97.5) (size 0.8) (drill 0.4) (layers F.Cu B.Cu) (net 1))
+  (segment (start 59.9 99.825) (end 62.225 97.5) (width 0.2032) (layer B.Cu) (net 1))
+  (segment (start 62.225 97.5) (end 67.9 97.5) (width 0.2032) (layer B.Cu) (net 1))
+  (segment (start 69.6708 96.5565) (end 70.624 96.5565) (width 0.2032) (layer B.Cu) (net 1))
+  (segment (start 69.409185 96.5565) (end 69.6708 96.5565) (width 0.2032) (layer B.Cu) (net 1))
+  (segment (start 68.465685 97.5) (end 69.409185 96.5565) (width 0.2032) (layer B.Cu) (net 1))
+  (segment (start 67.9 97.5) (end 68.465685 97.5) (width 0.2032) (layer B.Cu) (net 1))
   (segment (start 50.4 103.8282) (end 53.6718 107.1) (width 0.2032) (layer B.Cu) (net 2))
   (segment (start 50.4 103.075) (end 50.4 103.8282) (width 0.2032) (layer B.Cu) (net 2))
@@
   (segment (start 53.95 82.8625) (end 55.05 83.9625) (width 0.2032) (layer B.Cu) (net 26))
   (segment (start 53.95 77.02) (end 53.95 82.8625) (width 0.2032) (layer B.Cu) (net 26))
+  (segment (start 62 83.2375) (end 63.0125 84.25) (width 0.2032) (layer B.Cu) (net 27))
+  (segment (start 62 82.65) (end 62 83.2375) (width 0.2032) (layer B.Cu) (net 27))
+  (segment (start 73.124 86.7033) (end 73.124 87.6565) (width 0.2032) (layer B.Cu) (net 27))
+  (segment (start 73.124 85.949) (end 73.124 86.7033) (width 0.2032) (layer B.Cu) (net 27))
+  (segment (start 71.425 84.25) (end 73.124 85.949) (width 0.2032) (layer B.Cu) (net 27))
+  (segment (start 63.0125 84.25) (end 71.425 84.25) (width 0.2032) (layer B.Cu) (net 27))
+  (segment (start 60.601601 100.161769) (end 60.601601 99.693623) (width 0.2032) (layer B.Cu) (net 27))
+  (segment (start 60.236769 100.526601) (end 60.601601 100.161769) (width 0.2032) (layer B.Cu) (net 27))
+  (segment (start 58.854801 100.526601) (end 60.236769 100.526601) (width 0.2032) (layer B.Cu) (net 27))
+  (segment (start 56.6 99.375) (end 57.7032 99.375) (width 0.2032) (layer B.Cu) (net 27))
+  (segment (start 57.7032 99.375) (end 58.854801 100.526601) (width 0.2032) (layer B.Cu) (net 27))
   (segment (start 85.1065 97.3565) (end 82.024 97.3565) (width 0.2032) (layer B.Cu) (net 28))
   (segment (start 86.2 98.45) (end 85.1065 97.3565) (width 0.2032) (layer B.Cu) (net 28))

Commit message: Updated schematic
Parts:
- moved D1 28.4 mm to (105.4, 81.5)
- moved D4 25.6 mm to (124.5, 100.1)
- moved D3 2.78 mm to (105.4, 99.6), turned to 270 degrees
- moved D2 2.13 mm to (124.5, 81.3)
- moved C5 0.84 mm to (85.5, 89.3)
Routing:
- net ROW1: track 24.0 -> 0.00 mm
- net GND: track 144.2 -> 167.1 mm, vias 0 -> 4
- net Net-(R3-Pad2): track 19.6 -> 36.2 mm, vias 0 -> 2
- net +5V: track 42.5 -> 55.0 mm, vias 7 -> 0
- net Net-(D3-Pad2): track 7.71 -> 0.36 mm
- net Net-(C6-Pad1): track 0.00 -> 5.49 mm
- net (no net): vias 1 -> 0
Other:
- board size 82.1 x 38.8 mm -> 82.1 x 39 mm
