File: aidan pcb - copy.kicad_pcb (KiCad board)
At the start: 2 copper layers, 86 x 40 mm, 24 parts, among them SW1 SW_Push, U1 ATmega32U4-AU, Y1 16MHz

Commit message: final backup ocmpleted design
Parts:
- moved USB1 0.12 mm to (54.0, 72.5)
- moved MX4 0.06 mm to (116.5, 100.1)
Connections:
- U1 pad 27: ROW0 -> Net-(U1-Pad27)
- U1 pad 28: COL1 -> Net-(U1-Pad28)
- U1 pad 29: COL0 -> Net-(U1-Pad29)
- U1 pad 30: ROW1 -> Net-(U1-Pad30)
Routing:
- net ROW1: track 63.4 -> 15.5 mm, vias 2 -> 0
- net ROW0: track 40.6 -> 14.7 mm, vias 2 -> 0
- net COL0: track 50.0 -> 25.7 mm, vias 2 -> 0
- net COL1: track 40.1 -> 25.0 mm, vias 4 -> 2
- removed copper zone on B.Cu, net GND
Other:
- board size 86 x 40 mm -> 82.1 x 39 mm
- board text removed: "Prototype - 1"
- board text removed: "u/Pututski"
